File: hardware/task-controller/graphics.kicad_sch (KiCad schematic)
At the start: 4 parts

Commit message: preparing for production export
Parts:
- G3: footprint logo_silk:horn_logo_combined_7.500mm -> logo_silk:horn_logo_combined_5.000mm
Changed lines of the file:
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@@
 			)
 		)
-		(property "Footprint" "logo_silk:horn_logo_combined_7.500mm"
+		(property "Footprint" "logo_silk:horn_logo_combined_5.000mm"
 			(at 36.83 38.1 0)
 			(effects
@@
 		(at 30.48 24.13 0)
 		(unit 1)
-		(exclude_from_sim no)
+		(exclude_from_sim yes)
 		(in_bom no)
 		(on_board yes)
@@
 			(at 30.48 24.13 0)
 			(effects
-				(font
-					(size 1.27 1.27)
-				)
-				(hide yes)
-			)
-		)
-		(property "Sim.Enable" "0"
-			(at 30.48 24.13 0)
-			(effects
