File: hardware/task-controller/button_matrix.kicad_sch (KiCad schematic)
At the start: 56 parts, among them SW1 MATRIX, SW10 MATRIX, SW11 MATRIX, SW12 MATRIX, SW13 MATRIX, SW14 MATRIX, SW15 MATRIX, SW16 MATRIX, SW17 MATRIX, SW18 MATRIX, SW19 MATRIX, SW2 MATRIX, SW20 MATRIX, SW21 MATRIX, SW22 MATRIX, SW23 MATRIX, SW24 MATRIX, SW25 MATRIX, SW26 MATRIX, SW27 MATRIX, SW28 MATRIX, SW29 MATRIX, SW3 MATRIX, SW30 MATRIX, SW31 MATRIX, SW32 MATRIX, SW33 MATRIX, SW34 MATRIX, SW35 MATRIX, SW36 MATRIX, SW37 MATRIX, SW38 MATRIX, SW39 MATRIX, SW4 MATRIX, SW40 MATRIX, SW41 MATRIX, SW42 MATRIX, SW43 MATRIX, SW44 MATRIX, SW45 MATRIX, SW46 MATRIX, SW47 MATRIX, SW48 MATRIX, SW49 MATRIX, SW5 MATRIX, SW6 MATRIX, SW7 MATRIX, SW8 MATRIX, SW9 MATRIX

Commit message: most of rest of schematic
Other:
- note added: "Lay out in 3 columns of 16, with one spare (spare can be used as a reset all button or something)"
Changed lines of the file:
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@@
+		)
+	)
+	(text "Lay out in 3 columns of 16, with one spare\n(spare can be used as a reset all button or something)"
+		(exclude_from_sim no)
+		(at 201.168 22.098 0)
+		(effects
+			(font
+				(size 1.27 1.27)
+			)
 		)
 	)

Commit message: preparing for production export
Parts:
- SW1, SW10, SW11, SW12, SW13, SW14, SW15, SW16, SW17, SW18, SW19, SW2, SW20, SW21, SW22, SW23, SW24, SW25, SW26, SW27, SW28, SW29, SW3, SW30, SW31, SW32, SW33, SW34, SW35, SW36, SW37, SW38, SW39, SW4, SW40, SW41, SW42, SW43, SW44, SW45, SW46, SW47, SW48, SW49, SW5, SW6, SW7, SW8, SW9: LCSC Part # C64658 -> C160352
Changed lines of the file:
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@@
 			)
 		)
-		(property "LCSC Part #" "C64658"
+		(property "LCSC Part #" " C160352 "
 			(at 81.28 80.01 0)
 			(effects
@@
 			)
 		)
-		(property "LCSC Part #" "C64658"
+		(property "LCSC Part #" " C160352 "
 			(at 81.28 52.07 0)
 			(effects
@@
 			)
 		)
-		(property "LCSC Part #" "C64658"
+		(property "LCSC Part #" " C160352 "
 			(at 48.26 66.04 0)
 			(effects
@@
 			)
 		)
-		(property "LCSC Part #" "C64658"
+		(property "LCSC Part #" " C160352 "
 			(at 99.06 38.1 0)
 			(effects
@@
 			)
 		)
-		(property "LCSC Part #" "C64658"
+		(property "LCSC Part #" " C160352 "
 			(at 132.08 52.07 0)
 			(effects
@@
 			)
 		)
-		(property "LCSC Part #" "C64658"
+		(property "LCSC Part #" " C160352 "
 			(at 64.77 66.04 0)
 			(effects
@@
 			)
 		)
-		(property "LCSC Part #" "C64658"
+		(property "LCSC Part #" " C160352 "
 			(at 64.77 107.95 0)
 			(effects
@@
 			)
 		)
-		(property "LCSC Part #" "C64658"
+		(property "LCSC Part #" " C160352 "
 			(at 64.77 52.07 0)
 			(effects
@@
 			)
 		)
-		(property "LCSC Part #" "C64658"
+		(property "LCSC Part #" " C160352 "
 			(at 115.57 93.98 0)
 			(effects
@@
 			)
 		)
-		(property "LCSC Part #" "C64658"
+		(property "LCSC Part #" " C160352 "
 			(at 81.28 24.13 0)
 			(effects
@@
 			)
 		)
-		(property "LCSC Part #" "C64658"
+		(property "LCSC Part #" " C160352 "
 			(at 64.77 80.01 0)
 			(effects
@@
 			)
 		)
-		(property "LCSC Part #" "C64658"
+		(property "LCSC Part #" " C160352 "
 			(at 99.06 93.98 0)
 			(effects
@@
 			)
 		)
-		(property "LCSC Part #" "C64658"
+		(property "LCSC Part #" " C160352 "
 			(at 148.59 93.98 0)
 			(effects
@@
 			)
 		)
-		(property "LCSC Part #" "C64658"
+		(property "LCSC Part #" " C160352 "
 			(at 48.26 24.13 0)
 			(effects
@@
 			)
 		)
-		(property "LCSC Part #" "C64658"
+		(property "LCSC Part #" " C160352 "
 			(at 99.06 52.07 0)
 			(effects
@@
 			)
 		)
-		(property "LCSC Part #" "C64658"
+		(property "LCSC Part #" " C160352 "
 			(at 48.26 93.98 0)
 			(effects
@@
 			)
 		)
-		(property "LCSC Part #" "C64658"
+		(property "LCSC Part #" " C160352 "
 			(at 99.06 107.95 0)
 			(effects
@@
 			)
 		)
-		(property "LCSC Part #" "C64658"
+		(property "LCSC Part #" " C160352 "
 			(at 148.59 38.1 0)
 			(effects
@@
 			)
 		)
-		(property "LCSC Part #" "C64658"
+		(property "LCSC Part #" " C160352 "
 			(at 115.57 52.07 0)
 			(effects
@@
 			)
 		)
-		(property "LCSC Part #" "C64658"
+		(property "LCSC Part #" " C160352 "
 			(at 115.57 24.13 0)
 			(effects
@@
 			)
 		)
-		(property "LCSC Part #" "C64658"
+		(property "LCSC Part #" " C160352 "
 			(at 48.26 80.01 0)
 			(effects
@@
 			)
 		)
-		(property "LCSC Part #" "C64658"
+		(property "LCSC Part #" " C160352 "
 			(at 99.06 66.04 0)
 			(effects
@@
 			)
 		)
-		(property "LCSC Part #" "C64658"
+		(property "LCSC Part #" " C160352 "
 			(at 115.57 80.01 0)
 			(effects
@@
 			)
 		)
-		(property "LCSC Part #" "C64658"
+		(property "LCSC Part #" " C160352 "
 			(at 132.08 38.1 0)
 			(effects
@@
 			)
 		)
-		(property "LCSC Part #" "C64658"
+		(property "LCSC Part #" " C160352 "
 			(at 115.57 38.1 0)
 			(effects
@@
 			)
 		)
-		(property "LCSC Part #" "C64658"
+		(property "LCSC Part #" " C160352 "
 			(at 99.06 80.01 0)
 			(effects
@@
 			)
 		)
-		(property "LCSC Part #" "C64658"
+		(property "LCSC Part #" " C160352 "
 			(at 132.08 24.13 0)
 			(effects
@@
 			)
 		)
-		(property "LCSC Part #" "C64658"
+		(property "LCSC Part #" " C160352 "
 			(at 64.77 93.98 0)
 			(effects
@@
 			)
 		)
-		(property "LCSC Part #" "C64658"
+		(property "LCSC Part #" " C160352 "
 			(at 148.59 52.07 0)
 			(effects
@@
 			)
 		)
-		(property "LCSC Part #" "C64658"
+		(property "LCSC Part #" " C160352 "
 			(at 148.59 24.13 0)
 			(effects
@@
 			)
 		)
-		(property "LCSC Part #" "C64658"
+		(property "LCSC Part #" " C160352 "
 			(at 64.77 24.13 0)
 			(effects
@@
 			)
 		)
-		(property "LCSC Part #" "C64658"
+		(property "LCSC Part #" " C160352 "
 			(at 64.77 38.1 0)
 			(effects
@@
 			)
 		)
-		(property "LCSC Part #" "C64658"
+		(property "LCSC Part #" " C160352 "
 			(at 132.08 66.04 0)
 			(effects
@@
 			)
 		)
-		(property "LCSC Part #" "C64658"
+		(property "LCSC Part #" " C160352 "
 			(at 99.06 24.13 0)
 			(effects
@@
 			)
 		)
-		(property "LCSC Part #" "C64658"
+		(property "LCSC Part #" " C160352 "
 			(at 48.26 52.07 0)
 			(effects
@@
 			)
 		)
-		(property "LCSC Part #" "C64658"
+		(property "LCSC Part #" " C160352 "
 			(at 48.26 38.1 0)
 			(effects
@@
 			)
 		)
-		(property "LCSC Part #" "C64658"
+		(property "LCSC Part #" " C160352 "
 			(at 81.28 38.1 0)
 			(effects
@@
 			)
 		)
-		(property "LCSC Part #" "C64658"
+		(property "LCSC Part #" " C160352 "
 			(at 132.08 80.01 0)
 			(effects
@@
 			)
 		)
-		(property "LCSC Part #" "C64658"
+		(property "LCSC Part #" " C160352 "
 			(at 81.28 107.95 0)
 			(effects
@@
 			)
 		)
-		(property "LCSC Part #" "C64658"
+		(property "LCSC Part #" " C160352 "
 			(at 132.08 93.98 0)
 			(effects
@@
 			)
 		)
-		(property "LCSC Part #" "C64658"
+		(property "LCSC Part #" " C160352 "
 			(at 81.28 66.04 0)
 			(effects
@@
 			)
 		)
-		(property "LCSC Part #" "C64658"
+		(property "LCSC Part #" " C160352 "
 			(at 115.57 107.95 0)
 			(effects
@@
 			)
 		)
-		(property "LCSC Part #" "C64658"
+		(property "LCSC Part #" " C160352 "
 			(at 48.26 107.95 0)
 			(effects
@@
 			)
 		)
-		(property "LCSC Part #" "C64658"
+		(property "LCSC Part #" " C160352 "
 			(at 148.59 66.04 0)
 			(effects
@@
 			)
 		)
-		(property "LCSC Part #" "C64658"
+		(property "LCSC Part #" " C160352 "
 			(at 81.28 93.98 0)
 			(effects
@@
 			)
 		)
-		(property "LCSC Part #" "C64658"
+		(property "LCSC Part #" " C160352 "
 			(at 148.59 80.01 0)
 			(effects
@@
 			)
 		)
-		(property "LCSC Part #" "C64658"
+		(property "LCSC Part #" " C160352 "
 			(at 132.08 107.95 0)
 			(effects
@@
 			)
 		)
-		(property "LCSC Part #" "C64658"
+		(property "LCSC Part #" " C160352 "
 			(at 148.59 107.95 0)
 			(effects
@@
 			)
 		)
-		(property "LCSC Part #" "C64658"
+		(property "LCSC Part #" " C160352 "
 			(at 115.57 66.04 0)
 			(effects

Commit message: actual final production version
Parts:
- SW1, SW48, SW49: FT Rotation Offset (none) -> 180; LCSC Part # C160352 -> C2829150
- SW10: renamed from SW8; FT Rotation Offset (none) -> 180; LCSC Part # C160352 -> C2829150
- SW11: renamed from SW14; FT Rotation Offset (none) -> 180; LCSC Part # C160352 -> C2829150
- SW12: renamed from SW20; FT Rotation Offset (none) -> 180; LCSC Part # C160352 -> C2829150
- SW13: renamed from SW26; FT Rotation Offset (none) -> 180; LCSC Part # C160352 -> C2829150
- SW14: renamed from SW32; FT Rotation Offset (none) -> 180; LCSC Part # C160352 -> C2829150
- SW15: renamed from SW38; FT Rotation Offset (none) -> 180; LCSC Part # C160352 -> C2829150
- SW16: renamed from SW44; FT Rotation Offset (none) -> 180; LCSC Part # C160352 -> C2829150
- SW17: renamed from SW3; FT Rotation Offset (none) -> 180; LCSC Part # C160352 -> C2829150
- SW18: renamed from SW9; FT Rotation Offset (none) -> 180; LCSC Part # C160352 -> C2829150
- SW19: renamed from SW15; FT Rotation Offset (none) -> 180; LCSC Part # C160352 -> C2829150
- SW2: renamed from SW7; FT Rotation Offset (none) -> 180; LCSC Part # C160352 -> C2829150
- SW20: renamed from SW21; FT Rotation Offset (none) -> 180; LCSC Part # C160352 -> C2829150
- SW21: renamed from SW27; FT Rotation Offset (none) -> 180; LCSC Part # C160352 -> C2829150
- SW22: renamed from SW33; FT Rotation Offset (none) -> 180; LCSC Part # C160352 -> C2829150
- SW23: renamed from SW39; FT Rotation Offset (none) -> 180; LCSC Part # C160352 -> C2829150
- SW24: renamed from SW45; FT Rotation Offset (none) -> 180; LCSC Part # C160352 -> C2829150
- SW25: renamed from SW4; FT Rotation Offset (none) -> 180; LCSC Part # C160352 -> C2829150
- SW26: renamed from SW10; FT Rotation Offset (none) -> 180; LCSC Part # C160352 -> C2829150
- SW27: renamed from SW16; FT Rotation Offset (none) -> 180; LCSC Part # C160352 -> C2829150
- SW28: renamed from SW22; FT Rotation Offset (none) -> 180; LCSC Part # C160352 -> C2829150
- SW29: renamed from SW28; FT Rotation Offset (none) -> 180; LCSC Part # C160352 -> C2829150
- SW3: renamed from SW13; FT Rotation Offset (none) -> 180; LCSC Part # C160352 -> C2829150
- SW30: renamed from SW34; FT Rotation Offset (none) -> 180; LCSC Part # C160352 -> C2829150
- SW31: renamed from SW40; FT Rotation Offset (none) -> 180; LCSC Part # C160352 -> C2829150
- SW32: renamed from SW46; FT Rotation Offset (none) -> 180; LCSC Part # C160352 -> C2829150
- SW33: renamed from SW5; FT Rotation Offset (none) -> 180; LCSC Part # C160352 -> C2829150
- SW34: renamed from SW11; FT Rotation Offset (none) -> 180; LCSC Part # C160352 -> C2829150
- SW35: renamed from SW17; FT Rotation Offset (none) -> 180; LCSC Part # C160352 -> C2829150
- SW36: renamed from SW23; FT Rotation Offset (none) -> 180; LCSC Part # C160352 -> C2829150
- SW37: renamed from SW29; FT Rotation Offset (none) -> 180; LCSC Part # C160352 -> C2829150
- SW38: renamed from SW35; FT Rotation Offset (none) -> 180; LCSC Part # C160352 -> C2829150
- SW39: renamed from SW41; FT Rotation Offset (none) -> 180; LCSC Part # C160352 -> C2829150
- SW4: renamed from SW19; FT Rotation Offset (none) -> 180; LCSC Part # C160352 -> C2829150
- SW40: renamed from SW47; FT Rotation Offset (none) -> 180; LCSC Part # C160352 -> C2829150
- SW41: renamed from SW6; FT Rotation Offset (none) -> 180; LCSC Part # C160352 -> C2829150
- SW42: renamed from SW12; FT Rotation Offset (none) -> 180; LCSC Part # C160352 -> C2829150
- SW43: renamed from SW18; FT Rotation Offset (none) -> 180; LCSC Part # C160352 -> C2829150
- SW44: renamed from SW24; FT Rotation Offset (none) -> 180; LCSC Part # C160352 -> C2829150
- SW45: renamed from SW30; FT Rotation Offset (none) -> 180; LCSC Part # C160352 -> C2829150
- SW46: renamed from SW36; FT Rotation Offset (none) -> 180; LCSC Part # C160352 -> C2829150
- SW47: renamed from SW42; FT Rotation Offset (none) -> 180; LCSC Part # C160352 -> C2829150
- SW5: renamed from SW25; FT Rotation Offset (none) -> 180; LCSC Part # C160352 -> C2829150
- SW6: renamed from SW31; FT Rotation Offset (none) -> 180; LCSC Part # C160352 -> C2829150
- SW7: renamed from SW37; FT Rotation Offset (none) -> 180; LCSC Part # C160352 -> C2829150
- SW8: renamed from SW43; FT Rotation Offset (none) -> 180; LCSC Part # C160352 -> C2829150
- SW9: renamed from SW2; FT Rotation Offset (none) -> 180; LCSC Part # C160352 -> C2829150
- renumbered R25 to R1, R28 to R24, R24 to R3, R27 to R30, R26 to R31, R29 to R35, R30 to R5
