File: hardware/task-controller/mounting.kicad_sch (KiCad schematic)
At the start: 6 parts

Commit message: actual final production version
Parts:
- renumbered H3 to H1, H1 to H3, H6 to H4, H4 to H6
Changed lines of the file:
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@@
 		(dnp yes)
 		(fields_autoplaced yes)
-		(property "Reference" "H4"
+		(property "Reference" "H6"
 			(at 22.86 39.3699 0)
 			(effects
@@
 			(project "task-controller"
 				(path "/3313c311-f70a-45a8-bbf4-c9e4cbd18d5c/121f83e2-7284-4408-9524-8573a0418571"
-					(reference "H4")
+					(reference "H6")
 					(unit 1)
 				)
@@
 		(dnp yes)
 		(fields_autoplaced yes)
-		(property "Reference" "H3"
+		(property "Reference" "H1"
 			(at 71.12 19.0499 0)
 			(effects
@@
 			(project "task-controller"
 				(path "/3313c311-f70a-45a8-bbf4-c9e4cbd18d5c/121f83e2-7284-4408-9524-8573a0418571"
-					(reference "H3")
+					(reference "H1")
 					(unit 1)
 				)
@@
 		(dnp yes)
 		(fields_autoplaced yes)
-		(property "Reference" "H1"
+		(property "Reference" "H3"
 			(at 22.86 19.0499 0)
 			(effects
@@
 			(project ""
 				(path "/3313c311-f70a-45a8-bbf4-c9e4cbd18d5c/121f83e2-7284-4408-9524-8573a0418571"
-					(reference "H1")
+					(reference "H3")
 					(unit 1)
 				)
@@
 		(dnp yes)
 		(fields_autoplaced yes)
-		(property "Reference" "H6"
+		(property "Reference" "H4"
 			(at 71.12 39.3699 0)
 			(effects
@@
 			(project "task-controller"
 				(path "/3313c311-f70a-45a8-bbf4-c9e4cbd18d5c/121f83e2-7284-4408-9524-8573a0418571"
-					(reference "H6")
-					(unit 1)
-				)
+					(reference "H4")
+					(unit 1)
+				)
