File: hardware/task-controller/task-controller.kicad_sch (KiCad schematic)
At the start: 47 parts, among them J1 USB_C_Receptacle_USB2.0_16P, J6 Conn_01x06, J7 Conn_01x02, J8 SWD, J9 I2C, SW50 BOOTSEL, SW51 RST, U1 XC6206PxxxMR, U3 W25Q32JVSS, U4 RP2040, U5 FM24C64B, Y1 12MHz

Commit message: actual final production version
Parts:
- J1: FT Position Offset (none) -> -1.0795,0
- R22: renamed from R12; Cost (none) -> C64658; FT Rotation Offset (none) -> 180; LCSC Part # C64658 -> C2829150; now fitted
- U2: renamed from U4; FT Rotation Offset (none) -> 90
- renumbered C6 to C1, C16 to C10, C14 to C11, C11 to C12, C15 to C13, C9 to C14, C20 to C15, C7 to C17, C21 to C18, C8 to C2, C1 to C3, C2 to C4, C18 to C5, C10 to C6, C17 to C7, C12 to C8, C13 to C9, J9 to J2, J8 to J3, J7 to J5, R1 to R12, R4 to R13, R8 to R14, R10 to R15, R11 to R17, R21 to R19, R14 to R2, R3 to R20, R20 to R21, R22 to R25, R18 to R26, R19 to R27, R16 to R28, R9 to R4, R2 to R6, R15 to R7, SW51 to SW50, SW50 to SW51, U5 to U4
